Commit message: añadiendo paquete para uso de la camara web

File: autonomy/urdf/tracked_robot.xacro (robot description, xacro)
@@ -7,5 +7,5 @@
   <inertial>
     <origin xyz="-0.000697957365761748 -0.02693181329873898 -0.10360548608478944" rpy="0 0 0"/>
-    <mass value="189.21160692719502"/>
+    <mass value="25.21160692719502"/>
     <inertia ixx="8.567394" iyy="5.528814" izz="10.16907" ixy="0.002631" iyz="0.595537" ixz="0.007196"/>
   </inertial>
@@ -27,5 +27,5 @@
   <inertial>
     <origin xyz="0.017500185545245905 -0.15584208305997968 -0.17378022497017792" rpy="0 0 0"/>
-    <mass value="9.070297509831398"/>
+    <mass value="4.070297509831398"/>
     <inertia ixx="0.658697" iyy="0.100739" izz="0.583862" ixy="0.0" iyz="0.033262" ixz="0.0"/>
   </inertial>
@@ -42,5 +42,5 @@
       <mesh filename="package://autonomy/meshes/left_track_link_1.stl" scale="0.001 0.001 0.001"/>
     </geometry>
-    <surface>
+    <!-- <surface>
       <friction>
           <ode>
@@ -50,5 +50,5 @@
           </ode>
       </friction>
-    </surface>
+    </surface> -->
   </collision>
 </link>
@@ -56,5 +56,5 @@
   <inertial>
     <origin xyz="-0.017500185545247016 -0.15584208305997946 -0.17378022497017764" rpy="0 0 0"/>
-    <mass value="9.070297509831398"/>
+    <mass value="4.070297509831398"/>
     <inertia ixx="0.658697" iyy="0.100739" izz="0.583862" ixy="0.0" iyz="0.033262" ixz="-0.0"/>
   </inertial>
@@ -71,5 +71,5 @@
       <mesh filename="package://autonomy/meshes/right_track_link_1.stl" scale="0.001 0.001 0.001"/>
     </geometry>
-    <surface>
+    <!-- <surface>
       <friction>
           <ode>
@@ -79,5 +79,5 @@
           </ode>
       </friction>
-    </surface>
+    </surface> -->
   </collision>
 </link>
@@ -122,4 +122,6 @@
     <left_track>left_track_link_1</left_track>
     <right_track>right_track_link_1</right_track>
+    <!-- <steering_efficiency>0.5</steering_efficiency> -->
+    <!-- <tracks_separation>0.45</tracks_separation> -->
     <track_mu>2</track_mu>
     <track_mu2>0.5</track_mu2>
@@ -127,5 +129,5 @@
   <plugin filename="libKeysToCmdVelPlugin.so" name="keyboard_control">
     <publish_as_twist>true</publish_as_twist>
-    <cmd_vel_topic>~/simple_tracked/cmd_vel_twist</cmd_vel_topic>
+    <cmd_vel_topic>~/tracked_robot/cmd_vel_twist</cmd_vel_topic>
   </plugin>
 </gazebo>
